Commit message: chassis modification

File: description/gazebo_control.xacro (robot description, xacro)
@@ -4,6 +4,8 @@
         <plugin name="diff_drive" filename="libgazebo_ros_diff_drive.so">
             <!-- WHEEL INFORMATION -->
-            <left_joint>left_wheel_joint</left_joint>
-            <right_joint>right_wheel_joint</right_joint>
+            <left_joint>left_wheel_joint_1</left_joint>
+            <left_joint>left_wheel_joint_2</left_joint>
+            <right_joint>right_wheel_joint_2</right_joint>
+            <right_joint>right_wheel_joint_2</right_joint>
             <wheel_separation>0.35</wheel_separation>
             <wheel_diameter>0.1</wheel_diameter>

File: description/robot_core.xacro (robot description, xacro)
@@ -21,22 +21,22 @@
         <parent link="base_link"/>
         <child link="chassis"/>
-        <origin xyz="-0.1 0 0"/>
+        <origin xyz="0 0 0"/>
     </joint>
     <link name="chassis">
         <visual>
-            <origin xyz="0.15 0 0.075"/>
+            <origin xyz="0 0 0.075"/>
             <geometry>
-                <box size="0.3 0.3 0.15"/>
+                <box size="0.35 0.3 0.15"/>
             </geometry>
             <material name="white"/>
         </visual>
         <collision>
-            <origin xyz="0.15 0 0.075"/>
+            <origin xyz="0 0 0.075"/>
             <geometry>
-                <box size="0.3 0.3 0.15"/>
+                <box size="0.35 0.3 0.15"/>
             </geometry>
         </collision>
-        <xacro:inertial_box mass="0.5" x="0.3" y="0.3" z="0.15">
-            <origin xyz="0.15 0 0.075" rpy="0 0 0"/>
+        <xacro:inertial_box mass="0.5" x="0.35" y="0.3" z="0.15">
+            <origin xyz="0 0 0.075" rpy="0 0 0"/>
         </xacro:inertial_box>
     </link>
@@ -44,12 +44,12 @@
         <material>Gazebo/White</material>
     </gazebo>
-    <!-- LEFT WHEEL LINK -->
-    <joint name="left_wheel_joint" type="continuous">
+    <!-- LEFT WHEEL LINK 1-->
+    <joint name="left_wheel_joint_1" type="continuous">
         <parent link="base_link"/>
-        <child link="left_wheel"/>
-        <origin xyz="0 0.175 0" rpy="-${pi/2} 0 0" />
+        <child link="left_wheel_1"/>
+        <origin xyz="-0.1 0.175 0" rpy="-${pi/2} 0 0" />
         <axis xyz="0 0 1"/>
     </joint>
-    <link name="left_wheel">
+    <link name="left_wheel_1">
         <visual>
             <geometry>
@@ -67,15 +67,15 @@
         </xacro:inertial_cylinder>
     </link>
-    <gazebo reference="left_wheel">
+    <gazebo reference="left_wheel_1">
         <material>Gazebo/Blue</material>
     </gazebo>
-    <!-- RIGHT WHEEL LINK -->
-    <joint name="right_wheel_joint" type="continuous">
+    <!-- LEFT WHEEL LINK 2-->
+    <joint name="left_wheel_joint_2" type="continuous">
         <parent link="base_link"/>
-        <child link="right_wheel"/>
-        <origin xyz="0 -0.175 0" rpy="${pi/2} 0 0" />
-        <axis xyz="0 0 -1"/>
+        <child link="left_wheel_2"/>
+        <origin xyz="0.1 0.175 0" rpy="-${pi/2} 0 0" />
+        <axis xyz="0 0 1"/>
     </joint>
-    <link name="right_wheel">
+    <link name="left_wheel_2">
         <visual>
             <geometry>
@@ -93,8 +93,60 @@
         </xacro:inertial_cylinder>
     </link>
-    <gazebo reference="right_wheel">
+    <gazebo reference="left_wheel_2">
         <material>Gazebo/Blue</material>
     </gazebo>
-    <!-- CASTER WHEEL LINK -->
+    <!-- RIGHT WHEEL LINK 1 -->
+    <joint name="right_wheel_joint_1" type="continuous">
+        <parent link="base_link"/>
+        <child link="right_wheel_1"/>
+        <origin xyz="-0.1 -0.175 0" rpy="${pi/2} 0 0" />
+        <axis xyz="0 0 -1"/>
+    </joint>
+    <link name="right_wheel_1">
+        <visual>
+            <geometry>
+                <cylinder radius="0.05" length="0.04"/>
+            </geometry>
+            <material name="blue"/>
+        </visual>
+        <collision>
+            <geometry>
+                <cylinder radius="0.05" length="0.04"/>
+            </geometry>
+        </collision>
+        <xacro:inertial_cylinder mass="0.1" length="0.04" radius="0.05">
+            <origin xyz="0 0 0" rpy="0 0 0"/>
+        </xacro:inertial_cylinder>
+    </link>
+    <gazebo reference="right_wheel_1">
+        <material>Gazebo/Blue</material>
+    </gazebo>
+    <!-- RIGHT WHEEL LINK 2 -->
+    <joint name="right_wheel_joint_2" type="continuous">
+        <parent link="base_link"/>
+        <child link="right_wheel_2"/>
+        <origin xyz="0.1 -0.175 0" rpy="${pi/2} 0 0" />
+        <axis xyz="0 0 -1"/>
+    </joint>
+    <link name="right_wheel_2">
+        <visual>
+            <geometry>
+                <cylinder radius="0.05" length="0.04"/>
+            </geometry>
+            <material name="blue"/>
+        </visual>
+        <collision>
+            <geometry>
+                <cylinder radius="0.05" length="0.04"/>
+            </geometry>
+        </collision>
+        <xacro:inertial_cylinder mass="0.1" length="0.04" radius="0.05">
+            <origin xyz="0 0 0" rpy="0 0 0"/>
+        </xacro:inertial_cylinder>
+    </link>
+    <gazebo reference="right_wheel_2">
+        <material>Gazebo/Blue</material>
+    </gazebo>
+    <!-- CASTER WHEEL LINK
     <joint name="caster_wheel_joint" type="fixed">
         <parent link="chassis"/>
@@ -123,3 +175,4 @@
         <mu2 value="0.001"/>
     </gazebo>
+    -->
 </robot>

Commit message: opdate

File: description/gazebo_control.xacro (robot description, xacro)
@@ -4,8 +4,8 @@
         <plugin name="diff_drive" filename="libgazebo_ros_diff_drive.so">
             <!-- WHEEL INFORMATION -->
-            <left_joint>left_wheel_joint_1</left_joint>
-            <left_joint>left_wheel_joint_2</left_joint>
+            <left_joint>left_wheel_joint</left_joint>
+            <left_joint_2>left_wheel_joint</left_joint_2>
             <right_joint>right_wheel_joint_2</right_joint>
-            <right_joint>right_wheel_joint_2</right_joint>
+            <right_joint_2>right_wheel_joint_2</right_joint_2>
             <wheel_separation>0.35</wheel_separation>
             <wheel_diameter>0.1</wheel_diameter>

File: description/robot_core.xacro (robot description, xacro)
@@ -45,11 +45,11 @@
     </gazebo>
     <!-- LEFT WHEEL LINK 1-->
-    <joint name="left_wheel_joint_1" type="continuous">
+    <joint name="left_wheel_joint" type="continuous">
         <parent link="base_link"/>
-        <child link="left_wheel_1"/>
+        <child link="left_wheel"/>
         <origin xyz="-0.1 0.175 0" rpy="-${pi/2} 0 0" />
         <axis xyz="0 0 1"/>
     </joint>
-    <link name="left_wheel_1">
+    <link name="left_wheel">
         <visual>
             <geometry>
@@ -67,5 +67,5 @@
         </xacro:inertial_cylinder>
     </link>
-    <gazebo reference="left_wheel_1">
+    <gazebo reference="left_wheel">
         <material>Gazebo/Blue</material>
     </gazebo>
@@ -97,11 +97,11 @@
     </gazebo>
     <!-- RIGHT WHEEL LINK 1 -->
-    <joint name="right_wheel_joint_1" type="continuous">
+    <joint name="right_wheel_joint" type="continuous">
         <parent link="base_link"/>
-        <child link="right_wheel_1"/>
+        <child link="right_wheel"/>
         <origin xyz="-0.1 -0.175 0" rpy="${pi/2} 0 0" />
         <axis xyz="0 0 -1"/>
     </joint>
-    <link name="right_wheel_1">
+    <link name="right_wheel">
         <visual>
             <geometry>
@@ -119,5 +119,5 @@
         </xacro:inertial_cylinder>
     </link>
-    <gazebo reference="right_wheel_1">
+    <gazebo reference="right_wheel">
         <material>Gazebo/Blue</material>
     </gazebo>
